File: Flow_meter/sigfox_pcb.brd (EAGLE design)
At the start: 80.6 x 34 mm, 15 parts, among them J1 SMA-142-0701-801, U1 SFM11R2D

Commit message: First firmware micro Real
Parts:
- removed J3: (no value), CON_FLUJO:SAMTEC_SSW-106-01-T-S
- added J2: (no value), SSW-106-02-G_S_RA:CON6_1X6_TR_SSQ
Connections:
- net GND: now also J2.6; no longer J3.6
- net RST: now also J2.3; no longer J3.3
- net RX: now also J2.1; no longer J3.1
- net TX: now also J2.2; no longer J3.2
- net VDD: now also J2.5; no longer J3.5
- net WAKE_UP: now also J2.4; no longer J3.4
Routing:
- net TX: track 11.6 -> 12.5 mm
Changed lines of the file:
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@@
 <setting verticaltext="up"/>
 </settings>
-<grid distance="12" unitdist="mil" unit="mil" style="lines" multiple="1" display="no" altdistance="5" altunitdist="mil" altunit="mil"/>
+<grid distance="0.05" unitdist="mm" unit="mm" style="lines" multiple="1" display="no" altdistance="5" altunitdist="mil" altunit="mil"/>
 <layers>
 <layer number="1" name="Top" color="4" fill="1" visible="yes" active="yes"/>
@@
 <element name="H2" library="untitled" package="HOLE_3.0" value="HOLE-M3" x="77.6" y="31" smashed="yes"/>
 <element name="H4" library="untitled" package="HOLE_3.0" value="HOLE-M3" x="25" y="3" smashed="yes"/>
-<element name="J3" library="CON_FLUJO" package="SAMTEC_SSW-106-01-T-S" value="" x="69.088" y="3.81" smashed="yes">
-<attribute name="MPN" value="SSW-106-01-T-S" x="69.088" y="3.81" size="1.778" layer="27" display="off"/>
-<attribute name="NAME" x="58.2168" y="5.4102" size="2.0828" layer="25" ratio="10" rot="SR0"/>
-<attribute name="OC_FARNELL" value="1803421" x="69.088" y="3.81" size="1.778" layer="27" display="off"/>
-<attribute name="OC_NEWARK" value="11P9409" x="69.088" y="3.81" size="1.778" layer="27" display="off"/>
-<attribute name="PACKAGE" value="CONN .100 inch 6 POS SNGL ROW" x="69.088" y="3.81" size="1.778" layer="27" display="off"/>
-<attribute name="SUPPLIER" value="SAMTEC" x="69.088" y="3.81" size="1.778" layer="27" display="off"/>
-<attribute name="VALUE" x="56.9976" y="0.2286" size="2.0828" layer="27" ratio="10" rot="SR0"/>
+<element name="J2" library="SSW-106-02-G_S_RA" package="CON6_1X6_TR_SSQ" value="" x="62.6388" y="3.8124" smashed="yes">
+<attribute name="BUILT_BY" value="EMA_UL_Team" x="62.6388" y="3.8124" size="1.778" layer="27" display="off"/>
+<attribute name="MANUFACTURER_PART_NUMBER" value="SSW-106-02-G-S-RA" x="62.6388" y="3.8124" size="1.778" layer="27" display="off"/>
+<attribute name="NAME" x="59.3622" y="3.1774" size="1.27" layer="25" ratio="6" rot="SR0"/>
+<attribute name="VALUE" x="60.9116" y="3.1774" size="1.27" layer="21" ratio="6" rot="SR0"/>
+<attribute name="VENDOR" value="Samtec Inc" x="62.6388" y="3.8124" size="1.778" layer="27" display="off"/>
 </element>
 </elements>
@@
 <vertex x="80.6" y="34"/>
 </polygon>
-<contactref element="J3" pad="6"/>
 <wire x1="77.9399" y1="9.398" x2="77.9399" y2="9.652" width="0.1524" layer="16"/>
 <wire x1="77.9399" y1="9.398" x2="77.9399" y2="7.3279" width="0.3048" layer="16"/>
 <wire x1="77.9399" y1="7.3279" x2="74.422" y2="3.81" width="0.3048" layer="16"/>
-<wire x1="74.422" y1="3.81" x2="69.088" y2="3.81" width="0.3048" layer="16"/>
 <wire x1="47.5361" y1="6.604" x2="38.628321875" y2="6.604" width="0.3048" layer="16"/>
 <wire x1="38.628321875" y1="6.604" x2="34.510978125" y2="10.72134375" width="0.3048" layer="16"/>
@@
 <wire x1="53.0352" y1="14.6304" x2="53.0352" y2="10.7188" width="0.3048" layer="16"/>
 <wire x1="53.0352" y1="10.7188" x2="54.102" y2="9.652" width="0.3048" layer="16"/>
+<contactref element="J2" pad="6"/>
+<wire x1="74.422" y1="3.81" x2="68.9912" y2="3.81" width="0.3048" layer="16"/>
+<wire x1="68.9912" y1="3.81" x2="68.9888" y2="3.8124" width="0.3048" layer="16"/>
 </signal>
 <signal name="VDD">
@@
 <wire x1="50.7619" y1="14.224" x2="50.79" y2="14.224" width="0.3048" layer="16"/>
 <wire x1="50.79" y1="14.224" x2="52.324" y2="15.758" width="0.3048" layer="16"/>
-<contactref element="J3" pad="5"/>
 <wire x1="50.7619" y1="14.224" x2="47.625" y2="11.0871" width="0.3048" layer="16"/>
 <wire x1="47.625" y1="11.0871" x2="47.625" y2="10.5029" width="0.3048" layer="16"/>
@@
 <wire x1="49.276" y1="4.064" x2="52.07" y2="1.27" width="0.3048" layer="16"/>
 <wire x1="52.07" y1="1.27" x2="65.024" y2="1.27" width="0.3048" layer="16"/>
-<wire x1="65.024" y1="1.27" x2="66.548" y2="2.794" width="0.3048" layer="16"/>
-<wire x1="66.548" y1="2.794" x2="66.548" y2="3.81" width="0.3048" layer="16"/>
+<contactref element="J2" pad="5"/>
+<wire x1="65.024" y1="1.27" x2="66.4488" y2="2.6948" width="0.3048" layer="16"/>
+<wire x1="66.4488" y1="2.6948" x2="66.4488" y2="3.8124" width="0.3048" layer="16"/>
 </signal>
 <signal name="RST">
@@
 <contactref element="U1" pad="19"/>
 <wire x1="57.1109" y1="13.768" x2="57.3141" y2="13.5648" width="0.3048" layer="16"/>
-<contactref element="J3" pad="3"/>
 <wire x1="50.927" y1="10.5029" x2="50.927" y2="6.6929" width="0.3048" layer="16"/>
 <wire x1="50.927" y1="6.6929" x2="50.8381" y2="6.604" width="0.3048" layer="16"/>
 <wire x1="53.086" y1="2.032" x2="60.706" y2="2.032" width="0.3048" layer="16"/>
-<wire x1="60.706" y1="2.032" x2="61.468" y2="2.794" width="0.3048" layer="16"/>
-<wire x1="61.468" y1="2.794" x2="61.468" y2="3.81" width="0.3048" layer="16"/>
+<wire x1="60.706" y1="2.032" x2="61.368" y2="2.694" width="0.3048" layer="16"/>
 <wire x1="50.8381" y1="6.604" x2="50.8381" y2="4.3561" width="0.3048" layer="16"/>
 <wire x1="50.8381" y1="4.3561" x2="50.8" y2="4.318" width="0.3048" layer="16"/>
@@
 <wire x1="57.1109" y1="9.6129" x2="54.102" y2="6.604" width="0.3048" layer="16"/>
 <wire x1="54.102" y1="6.604" x2="50.8381" y2="6.604" width="0.3048" layer="16"/>
+<contactref element="J2" pad="3"/>
+<wire x1="61.3688" y1="3.8124" x2="61.368" y2="3.8116" width="0.3048" layer="16"/>
+<wire x1="61.368" y1="3.8116" x2="61.368" y2="2.694" width="0.3048" layer="16"/>
 </signal>
 <signal name="N$1">
@@
 <contactref element="U1" pad="13"/>
 <wire x1="63.7109" y1="13.768" x2="63.7109" y2="13.614321875" width="0.3048" layer="16"/>
-<contactref element="J3" pad="4"/>
-<wire x1="63.7109" y1="13.768" x2="63.7109" y2="4.1071" width="0.3048" layer="16"/>
-<wire x1="63.7109" y1="4.1071" x2="64.008" y2="3.81" width="0.3048" layer="16"/>
+<contactref element="J2" pad="4"/>
+<wire x1="63.9088" y1="3.8124" x2="63.7109" y2="4.0103" width="0.3048" layer="16"/>
+<wire x1="63.7109" y1="4.0103" x2="63.7109" y2="13.768" width="0.3048" layer="16"/>
 </signal>
 <signal name="TX">
 <contactref element="U1" pad="14"/>
-<contactref element="J3" pad="2"/>
 <wire x1="62.6109" y1="13.768" x2="62.6109" y2="11.0997" width="0.3048" layer="16"/>
 <wire x1="62.6109" y1="11.0997" x2="58.8264" y2="7.3152" width="0.3048" layer="16"/>
-<wire x1="58.8264" y1="7.3152" x2="58.8264" y2="3.9116" width="0.3048" layer="16"/>
-<wire x1="58.8264" y1="3.9116" x2="58.928" y2="3.81" width="0.3048" layer="16"/>
+<wire x1="58.8264" y1="7.3152" x2="58.8264" y2="4.85" width="0.3048" layer="16"/>
+<contactref element="J2" pad="2"/>
+<wire x1="58.8264" y1="4.85" x2="58.8264" y2="3.9116" width="0.3048" layer="16"/>
+<wire x1="58.8264" y1="4.85" x2="58.8288" y2="4.8476" width="0.3048" layer="16"/>
+<wire x1="58.8288" y1="4.8476" x2="58.8288" y2="3.8124" width="0.3048" layer="16"/>
 </signal>
 <signal name="RX">
 <contactref element="U1" pad="15"/>
-<contactref element="J3" pad="1"/>
 <wire x1="61.5109" y1="13.768" x2="61.5109" y2="12.1333" width="0.3048" layer="16"/>
-<wire x1="61.5109" y1="12.1333" x2="56.388" y2="7.0104" width="0.3048" layer="16"/>
-<wire x1="56.388" y1="7.0104" x2="56.388" y2="3.81" width="0.3048" layer="16"/>
+<contactref element="J2" pad="1"/>
+<wire x1="56.2888" y1="6.9112" x2="56.2888" y2="3.8124" width="0.3048" layer="16"/>
+<wire x1="61.5109" y1="12.1333" x2="56.2888" y2="6.9112" width="0.3048" layer="16"/>
 </signal>
 <signal name="N$12">
